File: board/board.kicad_sch (KiCad schematic)
At the start: 1 part

Commit message: initial
Parts:
- added J1: 003_power, on_edge:on_edge_2x05_device, symbol put_on_edge:003_power
- added J2: 003_power, on_edge:on_edge_2x05_host, symbol put_on_edge:003_power
- added R1, R2: 0R, Resistor_SMD:R_0603_1608Metric, symbol Device:R_Small
Connections:
- new net: J1.2 (GND), J2.2 (GND)
- new net: J1.3 (GND), J2.3 (GND)
- new net: J1.4 (GND), J2.4 (GND)
- new net: J1.5 (GND), J2.5 (GND)
- new net: J1.6 (1.2V), J2.6 (1.2V)
- new net: J1.7 (1.8V), J2.7 (1.8V)
- new net: J1.8 (2.5V), J2.8 (2.5V)
- new net: J1.9 (3.3V), R1.1
- new net: J2.9 (3.3V), R2.2
- new net ldo/3.3v: R1.2, R2.1
- new net ldo/5v: J1.10 (5V), J2.10 (5V)
- new net ldo/GND: J1.1 (GND), J2.1 (GND)
Other:
- sheet implementation renamed ldo
- sheet ldo: file implementation.kicad_sch -> ldo.kicad_sch
- sheet ldo ports: added 3.3v, 5v, GND; removed none
- note added: "Although power connectors are used this edgy can be connected to any connector which has pin 1 GND and pinns 9 and 10 as 5v and 3.3v"
- note removed: "Input connectors go here"
- note removed: "Output connectors go here"
Changed lines of the file:
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@@
 (kicad_sch (version 20211123) (generator eeschema)
   (paper "A4")
-  (text "Output connectors go here" (at 224.79 88.9 0)
+  (junction (at 167.64 130.81) (diameter 0) (color 0 0 0 0)
+  )
+  (junction (at 125.73 147.32) (diameter 0) (color 0 0 0 0)
+  )
+  (junction (at 115.57 133.35) (diameter 0) (color 0 0 0 0)
+  )
+  (wire (pts (xy 179.07 130.81) (xy 184.15 130.81))
+    (stroke (width 0) (type default) (color 0 0 0 0))
+  )
+  (wire (pts (xy 95.25 154.94) (xy 198.12 154.94))
+    (stroke (width 0) (type default) (color 0 0 0 0))
+  )
+  (wire (pts (xy 125.73 85.09) (xy 125.73 147.32))
+    (stroke (width 0) (type default) (color 0 0 0 0))
+  )
+  (wire (pts (xy 151.13 130.81) (xy 167.64 130.81))
+    (stroke (width 0) (type default) (color 0 0 0 0))
+  )
+  (wire (pts (xy 125.73 147.32) (xy 190.5 147.32))
+    (stroke (width 0) (type default) (color 0 0 0 0))
+  )
+  (wire (pts (xy 109.22 123.19) (xy 184.15 123.19))
+    (stroke (width 0) (type default) (color 0 0 0 0))
+  )
+  (wire (pts (xy 190.5 147.32) (xy 190.5 142.24))
+    (stroke (width 0) (type default) (color 0 0 0 0))
+  )
+  (wire (pts (xy 167.64 85.09) (xy 167.64 130.81))
+    (stroke (width 0) (type default) (color 0 0 0 0))
+  )
+  (wire (pts (xy 115.57 133.35) (xy 184.15 133.35))
+    (stroke (width 0) (type default) (color 0 0 0 0))
+  )
+  (wire (pts (xy 97.79 152.4) (xy 97.79 142.24))
+    (stroke (width 0) (type default) (color 0 0 0 0))
+  )
+  (wire (pts (xy 115.57 82.55) (xy 115.57 133.35))
+    (stroke (width 0) (type default) (color 0 0 0 0))
+  )
+  (wire (pts (xy 167.64 130.81) (xy 173.99 130.81))
+    (stroke (width 0) (type default) (color 0 0 0 0))
+  )
+  (wire (pts (xy 198.12 154.94) (xy 198.12 142.24))
+    (stroke (width 0) (type default) (color 0 0 0 0))
+  )
+  (wire (pts (xy 95.25 142.24) (xy 95.25 154.94))
+    (stroke (width 0) (type default) (color 0 0 0 0))
+  )
+  (wire (pts (xy 109.22 130.81) (xy 146.05 130.81))
+    (stroke (width 0) (type default) (color 0 0 0 0))
+  )
+  (wire (pts (xy 102.87 142.24) (xy 102.87 147.32))
+    (stroke (width 0) (type default) (color 0 0 0 0))
+  )
+  (wire (pts (xy 109.22 125.73) (xy 184.15 125.73))
+    (stroke (width 0) (type default) (color 0 0 0 0))
+  )
+  (wire (pts (xy 100.33 149.86) (xy 193.04 149.86))
+    (stroke (width 0) (type default) (color 0 0 0 0))
+  )
+  (wire (pts (xy 92.71 157.48) (xy 92.71 142.24))
+    (stroke (width 0) (type default) (color 0 0 0 0))
+  )
+  (wire (pts (xy 109.22 133.35) (xy 115.57 133.35))
+    (stroke (width 0) (type default) (color 0 0 0 0))
+  )
+  (wire (pts (xy 102.87 147.32) (xy 125.73 147.32))
+    (stroke (width 0) (type default) (color 0 0 0 0))
+  )
+  (wire (pts (xy 165.1 85.09) (xy 167.64 85.09))
+    (stroke (width 0) (type default) (color 0 0 0 0))
+  )
+  (wire (pts (xy 195.58 142.24) (xy 195.58 152.4))
+    (stroke (width 0) (type default) (color 0 0 0 0))
+  )
+  (wire (pts (xy 100.33 142.24) (xy 100.33 149.86))
+    (stroke (width 0) (type default) (color 0 0 0 0))
+  )
+  (wire (pts (xy 200.66 157.48) (xy 92.71 157.48))
+    (stroke (width 0) (type default) (color 0 0 0 0))
+  )
+  (wire (pts (xy 128.27 82.55) (xy 115.57 82.55))
+    (stroke (width 0) (type default) (color 0 0 0 0))
+  )
+  (wire (pts (xy 195.58 152.4) (xy 97.79 152.4))
+    (stroke (width 0) (type default) (color 0 0 0 0))
+  )
+  (wire (pts (xy 193.04 149.86) (xy 193.04 142.24))
+    (stroke (width 0) (type default) (color 0 0 0 0))
+  )
+  (wire (pts (xy 128.27 85.09) (xy 125.73 85.09))
+    (stroke (width 0) (type default) (color 0 0 0 0))
+  )
+  (wire (pts (xy 200.66 142.24) (xy 200.66 157.48))
+    (stroke (width 0) (type default) (color 0 0 0 0))
+  )
+  (wire (pts (xy 109.22 128.27) (xy 184.15 128.27))
+    (stroke (width 0) (type default) (color 0 0 0 0))
+  )
+  (text "Although power connectors are used this edgy can be connected to any connector which has pin 1 GND and pinns 9 and 10 as 5v and 3.3v"
+    (at 80.01 162.56 0)
     (effects (font (size 1.27 1.27)) (justify left bottom))
   )
-  (text "Input connectors go here" (at 49.53 88.9 0)
-    (effects (font (size 1.27 1.27)) (justify left bottom))
+  (symbol (lib_id "put_on_edge:003_power") (at 97.79 128.27 0) (mirror y) (unit 1)
+    (in_bom yes) (on_board yes)
+    (property "Reference" "J1" (id 0) (at 99.8982 111.379 0))
+    (property "Value" "003_power" (id 1) (at 99.8982 113.6904 0))
+    (property "Footprint" "on_edge:on_edge_2x05_device" (id 2) (at 90.17 111.76 0)
+      (effects (font (size 1.27 1.27)) hide)
+    )
+    (property "Datasheet" "" (id 3) (at 90.17 111.76 0)
+      (effects (font (size 1.27 1.27)) hide)
+    )
+    (pin "1")
+    (pin "10")
+    (pin "2")
+    (pin "3")
+    (pin "4")
+    (pin "5")
+    (pin "6")
+    (pin "7")
+    (pin "8")
+    (pin "9")
+  )
+  (symbol (lib_id "Device:R_Small") (at 176.53 130.81 90) (unit 1)
+    (in_bom yes) (on_board yes) (fields_autoplaced)
+    (property "Reference" "R2" (id 0) (at 176.53 124.46 90))
+    (property "Value" "0R" (id 1) (at 176.53 127 90))
+    (property "Footprint" "Resistor_SMD:R_0603_1608Metric" (id 2) (at 176.53 130.81 0)
+      (effects (font (size 1.27 1.27)) hide)
+    )
+    (property "Datasheet" "~" (id 3) (at 176.53 130.81 0)
+      (effects (font (size 1.27 1.27)) hide)
+    )
+    (pin "1")
+    (pin "2")
+  )
+  (symbol (lib_id "put_on_edge:003_power") (at 195.58 128.27 0) (unit 1)
+    (in_bom yes) (on_board yes)
+    (property "Reference" "J2" (id 0) (at 203.9112 127.9398 0)
+      (effects (font (size 1.27 1.27)) (justify left))
+    )
+    (property "Value" "003_power" (id 1) (at 203.9112 130.2512 0)
+      (effects (font (size 1.27 1.27)) (justify left))
+    )
+    (property "Footprint" "on_edge:on_edge_2x05_host" (id 2) (at 203.2 111.76 0)
+      (effects (font (size 1.27 1.27)) hide)
+    )
+    (property "Datasheet" "" (id 3) (at 203.2 111.76 0)
+      (effects (font (size 1.27 1.27)) hide)
+    )
+    (pin "1")
+    (pin "10")
+    (pin "2")
+    (pin "3")
+    (pin "4")
+    (pin "5")
+    (pin "6")
+    (pin "7")
+    (pin "8")
+    (pin "9")
   )
   (symbol (lib_id "Graphic:Logo_Open_Hardware_Small") (at 273.05 157.48 0) (unit 1)
@@
     )
   )
-  (sheet (at 114.3 72.39) (size 60.96 62.23) (fields_autoplaced)
+  (symbol (lib_id "Device:R_Small") (at 148.59 130.81 90) (unit 1)
+    (in_bom yes) (on_board yes) (fields_autoplaced)
+    (property "Reference" "R1" (id 0) (at 148.59 124.46 90))
+    (property "Value" "0R" (id 1) (at 148.59 127 90))
+    (property "Footprint" "Resistor_SMD:R_0603_1608Metric" (id 2) (at 148.59 130.81 0)
+      (effects (font (size 1.27 1.27)) hide)
+    )
+    (property "Datasheet" "~" (id 3) (at 148.59 130.81 0)
+      (effects (font (size 1.27 1.27)) hide)
+    )
+    (pin "1")
+    (pin "2")
+  )
+  (sheet (at 128.27 48.26) (size 36.83 39.37) (fields_autoplaced)
     (stroke (width 0.1524) (type solid) (color 0 0 0 0))
     (fill (color 0 0 0 0.0000))
-    (property "Sheet name" "implementation" (id 0) (at 114.3 71.6784 0)
+    (property "Sheet name" "ldo" (id 0) (at 128.27 47.5484 0)
       (effects (font (size 1.27 1.27)) (justify left bottom))
     )
-    (property "Sheet file" "implementation.kicad_sch" (id 1) (at 114.3 135.2046 0)
+    (property "Sheet file" "ldo.kicad_sch" (id 1) (at 128.27 88.2146 0)
       (effects (font (size 1.27 1.27)) (justify left top))
+    )
+    (pin "3.3v" input (at 165.1 85.09 0)
+      (effects (font (size 1.27 1.27)) (justify right))
+    )
+    (pin "GND" input (at 128.27 85.09 180)
+      (effects (font (size 1.27 1.27)) (justify left))
+    )
+    (pin "5v" input (at 128.27 82.55 180)
+      (effects (font (size 1.27 1.27)) (justify left))
     )
   )
@@
   )
   (symbol_instances
+    (path "/767ce4c6-0e55-4543-92f0-34cb8237a544/6bb5ca5c-7415-42a9-985b-09c137966385"
+      (reference "C1") (unit 1) (value "100nF") (footprint "Capacitor_SMD:C_0603_1608Metric")
+    )
+    (path "/767ce4c6-0e55-4543-92f0-34cb8237a544/bf4bdb44-1ce9-4d84-9dc1-aaed43a588f1"
+      (reference "C2") (unit 1) (value "1uF") (footprint "Capacitor_SMD:C_0603_1608Metric")
+    )
+    (path "/767ce4c6-0e55-4543-92f0-34cb8237a544/dd34b7a6-8448-4c7f-81f6-a8e49de64a92"
+      (reference "C3") (unit 1) (value "10uF") (footprint "Capacitor_SMD:C_0603_1608Metric")
+    )
+    (path "/767ce4c6-0e55-4543-92f0-34cb8237a544/196d1b70-9b37-46c7-aa9e-b41abaaa8c23"
+      (reference "C4") (unit 1) (value "1uF") (footprint "Capacitor_SMD:C_0603_1608Metric")
+    )
+    (path "/772494d9-828e-42c5-9167-72dce9f6c228"
+      (reference "J1") (unit 1) (value "003_power") (footprint "on_edge:on_edge_2x05_device")
+    )
+    (path "/abb769b5-66a4-4327-bef9-e53be3e8fbb3"
+      (reference "J2") (unit 1) (value "003_power") (footprint "on_edge:on_edge_2x05_host")
+    )
     (path "/b72b6f4a-7489-40f2-bb90-d75ae01aa368"
       (reference "LOGO1") (unit 1) (value "Logo_Open_Hardware_Small") (footprint "Symbol:OSHW-Symbol_6.7x6mm_SilkScreen")
     )
-  )
+    (path "/e18dc31f-35b1-4375-bab5-b0e8b60eedea"
+      (reference "R1") (unit 1) (value "0R") (footprint "Resistor_SMD:R_0603_1608Metric")
+    )
+    (path "/92ae8d01-1978-4392-bfed-2880750da076"
+      (reference "R2") (unit 1) (value "0R") (footprint "Resistor_SMD:R_0603_1608Metric")
+    )
+    (path "/767ce4c6-0e55-4543-92f0-34cb8237a544/673b772a-b7c6-480f-97cf-a61f161efbae"
+      (reference "U1") (unit 1) (value "TC1017") (footprint "Package_TO_SOT_SMD:SOT-23-5")
+    )
+  )
